File: Peak-And-Hold/Peak-And-Hold.kicad_sch (KiCad schematic)
At the start: 31 parts, among them Q1 2N6044, Q2 2N6044, Q3 2N6044, Q4 2N6044, Q5 TIP42C, U1 LM1949N_NOPB, U2 LM1949N_NOPB, U3 LM1949N_NOPB, U4 LM1949N_NOPB

Commit message: added plugs
Parts:
- added J1, J2: 39301080, Connector_Molex:Molex_Mini-Fit_Jr_5569-08A2_2x04_P4.20mm_Horizontal, symbol Simon:39301080
Connections:
- net 5v: now also J1.5, J2.8
- net GND: now also J1.8, J2.5; no longer U1.6 (SUPPLY_GND), U2.6 (SUPPLY_GND), U3.6 (SUPPLY_GND), U4.6 (SUPPLY_GND)
- net INJ1: now also J1.2
- net INJ1OUT: now also J1.1
- net INJ2: now also J1.3
- net INJ2OUT: now also J1.4
- net INJ3: now also J2.2
- net INJ3OUT: now also J2.1
- net INJ4: now also J2.3
- net INJ4OUT: now also J2.4
- new net LoGND: J1.6, J1.7, J2.6, J2.7, U1.6 (SUPPLY_GND), U2.6 (SUPPLY_GND), U3.6 (SUPPLY_GND), U4.6 (SUPPLY_GND)

Commit message: finished off
Connections:
- net 5v: now also J1.8; no longer J1.5
- net GND: now also J1.5; no longer J1.8
Other:
- moved on the sheet: D5, Q5, R9

Commit message: Fabrication Ready
Parts:
- D5: value 1SMA4748A -> 1SMA4754A
Changed lines of the file:
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@@
       (effects (font (size 1.27 1.27)) (justify left))
     )
-    (property "Value" "1SMA4748A" (id 1) (at 233.68 72.3899 90)
+    (property "Value" "1SMA4754A" (id 1) (at 233.68 72.3899 90)
       (effects (font (size 1.27 1.27)) (justify left))
     )
@@
     )
     (path "/3f8a9cf3-9069-472a-b579-008b7c7761ab"
-      (reference "D5") (unit 1) (value "1SMA4748A") (footprint "Diode_SMD:D_SMA")
+      (reference "D5") (unit 1) (value "1SMA4754A") (footprint "Diode_SMD:D_SMA")
     )
     (path "/c98d36b8-9034-4cc3-842e-e855c4c8d2d2"
